Commit message: Biped visible and controllable in Gazebo (ros2_control working)

File: src/my_robot_description/urdf/my_biped.urdf.xacro (robot description, xacro)
@@ -2,121 +2,154 @@
 <robot name="my_biped" xmlns:xacro="http://www.ros.org/wiki/xacro">
 <xacro:arg name="controllers_yaml" default=""/>
-  <!-- ================= -->
-  <!-- Inertia macro -->
-  <!-- ================= -->
-  <xacro:macro name="box_inertia" params="m x y z">
-    <inertial>
-      <mass value="${m}"/>
-      <inertia
-        ixx="${m*(y*y+z*z)/12}"
-        iyy="${m*(x*x+z*z)/12}"
-        izz="${m*(x*x+y*y)/12}"
-        ixy="0" ixz="0" iyz="0"/>
-    </inertial>
-  </xacro:macro>
-  <!-- ================= -->
-  <!-- BASE (ROOT) -->
-  <!-- ================= -->
-  <link name="base_link">
-    <xacro:box_inertia m="6.0" x="0.3" y="0.2" z="0.1"/>
+<material name="red">
+  <color rgba="0.8 0.1 0.1 1"/>
+</material>
+<material name="green">
+  <color rgba="0.2 0.8 0.2 1"/>
+</material>
+<material name="blue">
+  <color rgba="0.2 0.2 0.8 1"/>
+</material>
+<material name="gray">
+  <color rgba="0.6 0.6 0.6 1"/>
+</material>
+<!-- ================= -->
+<!-- Inertia macro -->
+<!-- ================= -->
+<xacro:macro name="box_inertia" params="m x y z">
+  <inertial>
+    <mass value="${m}"/>
+    <inertia
+      ixx="${m*(y*y+z*z)/12}"
+      iyy="${m*(x*x+z*z)/12}"
+      izz="${m*(x*x+y*y)/12}"
+      ixy="0" ixz="0" iyz="0"/>
+  </inertial>
+</xacro:macro>
+<!-- ================= -->
+<!-- BASE (ROOT) -->
+<!-- ================= -->
+<link name="base_link">
+  <xacro:box_inertia m="6.0" x="0.3" y="0.2" z="0.1"/>
+  <visual>
+    <origin xyz="0 0 0.05" rpy="0 0 0"/>
+    <geometry>
+      <box size="0.3 0.2 0.1"/>
+    </geometry>
+    <material name="red"/>
+  </visual>
+  <collision>
+    <origin xyz="0 0 0.05" rpy="0 0 0"/>
+    <geometry>
+      <box size="0.3 0.2 0.1"/>
+    </geometry>
+  </collision>
+</link>
+<gazebo reference="base_link">
+  <material>Gazebo/Red</material>
+</gazebo>
+<!-- ================= -->
+<!-- LEG MACRO -->
+<!-- ================= -->
+<xacro:macro name="leg" params="side y">
+  <!-- THIGH -->
+  <link name="${side}_thigh">
+    <xacro:box_inertia m="1.5" x="0.05" y="0.05" z="0.25"/>
     <visual>
-      <geometry><box size="0.3 0.2 0.1"/></geometry>
+      <origin xyz="0 0 0" rpy="0 0 0"/>
+      <geometry>
+        <box size="0.05 0.05 0.25"/>
+      </geometry>
+      <material name="green"/>
     </visual>
     <collision>
-      <geometry><box size="0.3 0.2 0.1"/></geometry>
+      <origin xyz="0 0 0" rpy="0 0 0"/>
+      <geometry>
+        <box size="0.05 0.05 0.25"/>
+      </geometry>
     </collision>
   </link>
-  <gazebo reference="base_link">
-    <material>Gazebo/Red</material>
-  </gazebo>
-   <!-- ================= -->
-  <!-- LEG MACRO -->
-  <!-- ================= -->
-  <xacro:macro name="leg" params="side y">
-    <!-- THIGH -->
-    <link name="${side}_thigh">
-      <xacro:box_inertia m="1.5" x="0.05" y="0.05" z="0.25"/>
-      <visual>
-        <geometry>
-          <box size="0.05 0.05 0.25"/>
-        </geometry>
-      </visual>
-      <collision>
-        <geometry>
-          <box size="0.05 0.05 0.25"/>
-        </geometry>
-      </collision>
-    </link>
-    <gazebo reference="${side}_thigh">
-      <material>Gazebo/Green</material>
-    </gazebo>
-    <joint name="${side}_hip" type="revolute">
-      <parent link="base_link"/>
-      <child link="${side}_thigh"/>
-      <origin xyz="0.05 ${y} -0.05"/>
-      <axis xyz="1 0 0"/>
-      <limit lower="-1.0" upper="1.0" effort="40" velocity="4"/>
-      <dynamics damping="10" friction="3"/>
-    </joint>
-    <!-- SHIN -->
-    <link name="${side}_shin">
-      <xacro:box_inertia m="1.0" x="0.04" y="0.04" z="0.25"/>
-      <visual>
-        <geometry>
-          <box size="0.04 0.04 0.25"/>
-        </geometry>
-      </visual>
-      <collision>
-        <geometry>
-          <box size="0.04 0.04 0.25"/>
-        </geometry>
-      </collision>
-    </link>
-    <gazebo reference="${side}_shin">
-      <material>Gazebo/Blue</material>
-    </gazebo>
-    <joint name="${side}_knee" type="revolute">
-      <parent link="${side}_thigh"/>
-      <child link="${side}_shin"/>
-      <origin xyz="0 0 -0.25"/>
-      <axis xyz="1 0 0"/>
-      <limit lower="0.0" upper="2.2" effort="40" velocity="4"/>
-      <dynamics damping="10" friction="3"/>
-    </joint>
-    <!-- FOOT -->
-    <link name="${side}_foot">
-      <xacro:box_inertia m="0.8" x="0.08" y="0.12" z="0.04"/>
-      <visual>
-        <origin xyz="0 0 -0.02"/>
-        <geometry>
-          <box size="0.08 0.12 0.04"/>
-        </geometry>
-      </visual>
-      <collision>
-        <origin xyz="0 0 -0.02"/>
-        <geometry>
-          <box size="0.08 0.12 0.04"/>
-        </geometry>
-      </collision>
-    </link>
-    <gazebo reference="${side}_foot">
-      <material>Gazebo/Gray</material>
-      <mu1>2.0</mu1>
-      <mu2>2.0</mu2>
-    </gazebo>
-    <joint name="${side}_ankle" type="revolute">
-      <parent link="${side}_shin"/>
-      <child link="${side}_foot"/>
-      <origin xyz="0 0 -0.25"/>
-      <axis xyz="1 0 0"/>
-      <limit lower="-0.6" upper="0.6" effort="30" velocity="4"/>
-      <dynamics damping="10" friction="3"/>
-    </joint>
-  </xacro:macro>
-  <!-- ================= -->
-  <!-- LEGS -->
-  <!-- ================= -->
-  <xacro:leg side="left"  y="0.06"/>
-  <xacro:leg side="right" y="-0.06"/>
+  <joint name="${side}_hip" type="revolute">
+    <parent link="base_link"/>
+    <child link="${side}_thigh"/>
+    <origin xyz="0.05 ${y} -0.05"/>
+    <axis xyz="1 0 0"/>
+    <limit lower="-1.0" upper="1.0" effort="40" velocity="4"/>
+    <dynamics damping="10" friction="3"/>
+  </joint>
+  <!-- SHIN -->
+  <link name="${side}_shin">
+    <xacro:box_inertia m="1.0" x="0.04" y="0.04" z="0.25"/>
+    <visual>
+      <origin xyz="0 0 0" rpy="0 0 0"/>
+      <geometry>
+        <box size="0.04 0.04 0.25"/>
+      </geometry>
+      <material name="blue"/>
+    </visual>
+    <collision>
+      <origin xyz="0 0 0" rpy="0 0 0"/>
+      <geometry>
+        <box size="0.04 0.04 0.25"/>
+      </geometry>
+    </collision>
+  </link>
+  <joint name="${side}_knee" type="revolute">
+    <parent link="${side}_thigh"/>
+    <child link="${side}_shin"/>
+    <origin xyz="0 0 -0.25"/>
+    <axis xyz="1 0 0"/>
+    <limit lower="0.0" upper="2.2" effort="40" velocity="4"/>
+    <dynamics damping="10" friction="3"/>
+  </joint>
+  <gazebo reference="left_thigh">
+  <material>Gazebo/Green</material>
+</gazebo>
+<gazebo reference="right_thigh">
+  <material>Gazebo/Green</material>
+</gazebo>
+  <!-- FOOT -->
+  <link name="${side}_foot">
+    <xacro:box_inertia m="0.8" x="0.08" y="0.12" z="0.04"/>
+    <visual>
+      <origin xyz="0 0 -0.02" rpy="0 0 0"/>
+      <geometry>
+        <box size="0.08 0.12 0.04"/>
+      </geometry>
+      <material name="gray"/>
+    </visual>
+    <collision>
+      <origin xyz="0 0 -0.02" rpy="0 0 0"/>
+      <geometry>
+        <box size="0.08 0.12 0.04"/>
+      </geometry>
+    </collision>
+  </link>
+  <joint name="${side}_ankle" type="revolute">
+    <parent link="${side}_shin"/>
+    <child link="${side}_foot"/>
+    <origin xyz="0 0 -0.25"/>
+    <axis xyz="1 0 0"/>
+    <limit lower="-0.6" upper="0.6" effort="30" velocity="4"/>
+    <dynamics damping="10" friction="3"/>
+  </joint>
+  <gazebo reference="left_shin">
+  <material>Gazebo/Blue</material>
+</gazebo>
+<gazebo reference="right_shin">
+  <material>Gazebo/Blue</material>
+</gazebo>
+<gazebo reference="left_foot">
+  <material>Gazebo/Grey</material>
+</gazebo>
+<gazebo reference="right_foot">
+  <material>Gazebo/Grey</material>
+</gazebo>
+</xacro:macro>
+<!-- ================= -->
+<!-- LEGS -->
+<!-- ================= -->
+<xacro:leg side="left"  y="0.06"/>
+<xacro:leg side="right" y="-0.06"/>
   <!-- =============================== -->
   <!-- ROS 2 CONTROL SYSTEM -->
@@ -157,7 +190,4 @@
     </joint>
   </ros2_control>
-  <!-- =============================== -->
-  <!-- Gazebo Classic ros2_control -->
-  <!-- =============================== -->
     <!-- =============================== -->
   <!-- Gazebo Classic ros2_control -->

Commit message: Fix biped geometry and switch to joint_trajectory_controller (stable kinematics)

File: src/my_robot_description/urdf/my_biped.urdf.xacro (robot description, xacro)
@@ -1,155 +1,125 @@
 <?xml version="1.0"?>
 <robot name="my_biped" xmlns:xacro="http://www.ros.org/wiki/xacro">
-<xacro:arg name="controllers_yaml" default=""/>
-<material name="red">
-  <color rgba="0.8 0.1 0.1 1"/>
-</material>
-<material name="green">
-  <color rgba="0.2 0.8 0.2 1"/>
-</material>
-<material name="blue">
-  <color rgba="0.2 0.2 0.8 1"/>
-</material>
-<material name="gray">
-  <color rgba="0.6 0.6 0.6 1"/>
-</material>
-<!-- ================= -->
-<!-- Inertia macro -->
-<!-- ================= -->
-<xacro:macro name="box_inertia" params="m x y z">
-  <inertial>
-    <mass value="${m}"/>
-    <inertia
-      ixx="${m*(y*y+z*z)/12}"
-      iyy="${m*(x*x+z*z)/12}"
-      izz="${m*(x*x+y*y)/12}"
-      ixy="0" ixz="0" iyz="0"/>
-  </inertial>
-</xacro:macro>
-<!-- ================= -->
-<!-- BASE (ROOT) -->
-<!-- ================= -->
-<link name="base_link">
-  <xacro:box_inertia m="6.0" x="0.3" y="0.2" z="0.1"/>
-  <visual>
-    <origin xyz="0 0 0.05" rpy="0 0 0"/>
-    <geometry>
-      <box size="0.3 0.2 0.1"/>
-    </geometry>
-    <material name="red"/>
-  </visual>
-  <collision>
-    <origin xyz="0 0 0.05" rpy="0 0 0"/>
-    <geometry>
-      <box size="0.3 0.2 0.1"/>
-    </geometry>
-  </collision>
-</link>
-<gazebo reference="base_link">
-  <material>Gazebo/Red</material>
-</gazebo>
-<!-- ================= -->
-<!-- LEG MACRO -->
-<!-- ================= -->
-<xacro:macro name="leg" params="side y">
-  <!-- THIGH -->
-  <link name="${side}_thigh">
-    <xacro:box_inertia m="1.5" x="0.05" y="0.05" z="0.25"/>
+  <!-- Path to controllers yaml -->
+  <xacro:arg name="controllers_yaml"
+             default="$(find my_robot_description)/config/controllers.yaml"/>
+  <!-- ================= -->
+  <!-- Materials -->
+  <!-- ================= -->
+  <material name="red"><color rgba="0.8 0.1 0.1 1"/></material>
+  <material name="green"><color rgba="0.2 0.8 0.2 1"/></material>
+  <material name="blue"><color rgba="0.2 0.2 0.8 1"/></material>
+  <material name="gray"><color rgba="0.6 0.6 0.6 1"/></material>
+  <!-- ================= -->
+  <!-- Inertia macro -->
+  <!-- ================= -->
+  <xacro:macro name="box_inertia" params="m x y z">
+    <inertial>
+      <mass value="${m}"/>
+      <inertia
+        ixx="${m*(y*y+z*z)/12}"
+        iyy="${m*(x*x+z*z)/12}"
+        izz="${m*(x*x+y*y)/12}"
+        ixy="0" ixz="0" iyz="0"/>
+    </inertial>
+  </xacro:macro>
+  <!-- ================= -->
+  <!-- BASE (ROOT) -->
+  <!-- ================= -->
+  <link name="base_link">
+    <xacro:box_inertia m="6.0" x="0.12" y="0.22" z="0.12"/>
     <visual>
-      <origin xyz="0 0 0" rpy="0 0 0"/>
-      <geometry>
-        <box size="0.05 0.05 0.25"/>
-      </geometry>
-      <material name="green"/>
+      <geometry><box size="0.12 0.22 0.12"/></geometry>
+      <material name="red"/>
     </visual>
     <collision>
-      <origin xyz="0 0 0" rpy="0 0 0"/>
-      <geometry>
-        <box size="0.05 0.05 0.25"/>
-      </geometry>
+      <geometry><box size="0.12 0.22 0.12"/></geometry>
     </collision>
   </link>
-  <joint name="${side}_hip" type="revolute">
-    <parent link="base_link"/>
-    <child link="${side}_thigh"/>
-    <origin xyz="0.05 ${y} -0.05"/>
-    <axis xyz="1 0 0"/>
-    <limit lower="-1.0" upper="1.0" effort="40" velocity="4"/>
-    <dynamics damping="10" friction="3"/>
-  </joint>
-  <!-- SHIN -->
-  <link name="${side}_shin">
-    <xacro:box_inertia m="1.0" x="0.04" y="0.04" z="0.25"/>
-    <visual>
-      <origin xyz="0 0 0" rpy="0 0 0"/>
-      <geometry>
-        <box size="0.04 0.04 0.25"/>
-      </geometry>
-      <material name="blue"/>
-    </visual>
-    <collision>
-      <origin xyz="0 0 0" rpy="0 0 0"/>
-      <geometry>
-        <box size="0.04 0.04 0.25"/>
-      </geometry>
-    </collision>
-  </link>
-  <joint name="${side}_knee" type="revolute">
-    <parent link="${side}_thigh"/>
-    <child link="${side}_shin"/>
-    <origin xyz="0 0 -0.25"/>
-    <axis xyz="1 0 0"/>
-    <limit lower="0.0" upper="2.2" effort="40" velocity="4"/>
-    <dynamics damping="10" friction="3"/>
-  </joint>
-  <gazebo reference="left_thigh">
-  <material>Gazebo/Green</material>
-</gazebo>
-<gazebo reference="right_thigh">
-  <material>Gazebo/Green</material>
-</gazebo>
-  <!-- FOOT -->
-  <link name="${side}_foot">
-    <xacro:box_inertia m="0.8" x="0.08" y="0.12" z="0.04"/>
-    <visual>
-      <origin xyz="0 0 -0.02" rpy="0 0 0"/>
-      <geometry>
-        <box size="0.08 0.12 0.04"/>
-      </geometry>
-      <material name="gray"/>
-    </visual>
-    <collision>
-      <origin xyz="0 0 -0.02" rpy="0 0 0"/>
-      <geometry>
-        <box size="0.08 0.12 0.04"/>
-      </geometry>
-    </collision>
-  </link>
-  <joint name="${side}_ankle" type="revolute">
-    <parent link="${side}_shin"/>
-    <child link="${side}_foot"/>
-    <origin xyz="0 0 -0.25"/>
-    <axis xyz="1 0 0"/>
-    <limit lower="-0.6" upper="0.6" effort="30" velocity="4"/>
-    <dynamics damping="10" friction="3"/>
-  </joint>
-  <gazebo reference="left_shin">
-  <material>Gazebo/Blue</material>
-</gazebo>
-<gazebo reference="right_shin">
-  <material>Gazebo/Blue</material>
-</gazebo>
-<gazebo reference="left_foot">
-  <material>Gazebo/Grey</material>
-</gazebo>
-<gazebo reference="right_foot">
-  <material>Gazebo/Grey</material>
-</gazebo>
-</xacro:macro>
-<!-- ================= -->
-<!-- LEGS -->
-<!-- ================= -->
-<xacro:leg side="left"  y="0.06"/>
-<xacro:leg side="right" y="-0.06"/>
+  <gazebo reference="base_link"><material>Gazebo/Red</material></gazebo>
+  <!-- ================= -->
+  <!-- LEG MACRO -->
+  <!-- ================= -->
+  <xacro:macro name="leg" params="side y">
+    <!-- THIGH -->
+    <link name="${side}_thigh">
+      <xacro:box_inertia m="1.5" x="0.05" y="0.05" z="0.25"/>
+      <visual>
+        <origin xyz="0 0 -0.125"/>
+        <geometry><box size="0.05 0.05 0.25"/></geometry>
+        <material name="green"/>
+      </visual>
+      <collision>
+        <origin xyz="0 0 -0.125"/>
+        <geometry><box size="0.05 0.05 0.25"/></geometry>
+      </collision>
+    </link>
+    <joint name="${side}_hip" type="revolute">
+      <parent link="base_link"/>
+      <child link="${side}_thigh"/>
+      <origin xyz="0 ${y} 0"/>
+      <axis xyz="0 1 0"/>
+      <limit lower="-1.0" upper="1.0" effort="40" velocity="3"/>
+      <dynamics damping="2.0" friction="0.5"/>
+    </joint>
+    <!-- SHIN -->
+    <link name="${side}_shin">
+      <xacro:box_inertia m="1.0" x="0.045" y="0.045" z="0.25"/>
+      <visual>
+        <origin xyz="0 0 -0.125"/>
+        <geometry><box size="0.045 0.045 0.25"/></geometry>
+        <material name="blue"/>
+      </visual>
+      <collision>
+        <origin xyz="0 0 -0.125"/>
+        <geometry><box size="0.045 0.045 0.25"/></geometry>
+      </collision>
+    </link>
+    <joint name="${side}_knee" type="revolute">
+      <parent link="${side}_thigh"/>
+      <child link="${side}_shin"/>
+      <origin xyz="0 0 -0.25"/>
+      <axis xyz="0 1 0"/>
+      <limit lower="0.0" upper="2.2" effort="40" velocity="3"/>
+      <dynamics damping="3.0" friction="0.8"/>
+    </joint>
+    <!-- FOOT -->
+    <link name="${side}_foot">
+      <xacro:box_inertia m="0.8" x="0.12" y="0.08" z="0.04"/>
+      <visual>
+        <origin xyz="0 0 -0.02"/>
+        <geometry><box size="0.12 0.08 0.04"/></geometry>
+        <material name="gray"/>
+      </visual>
+      <collision>
+        <origin xyz="0 0 -0.02"/>
+        <geometry><box size="0.12 0.08 0.04"/></geometry>
+      </collision>
+    </link>
+    <joint name="${side}_ankle" type="revolute">
+      <parent link="${side}_shin"/>
+      <child link="${side}_foot"/>
+      <origin xyz="0.04 0 -0.25"/>
+      <axis xyz="0 1 0"/>
+      <limit lower="-0.6" upper="0.6" effort="30" velocity="3"/>
+      <dynamics damping="1.5" friction="0.4"/>
+    </joint>
+    <!-- Gazebo colors -->
+    <gazebo reference="${side}_thigh"><material>Gazebo/Green</material></gazebo>
+    <gazebo reference="${side}_shin"><material>Gazebo/Blue</material></gazebo>
+    <gazebo reference="${side}_foot"><material>Gazebo/Grey</material></gazebo>
+    <!-- FOOT CONTACT -->
+    <gazebo reference="${side}_foot">
+      <mu1>1.0</mu1>
+      <mu2>1.0</mu2>
+      <kp>80000</kp>
+      <kd>150</kd>
+    </gazebo>
+  </xacro:macro>
+  <!-- ================= -->
+  <!-- LEGS -->
+  <!-- ================= -->
+  <xacro:leg side="left"  y="0.06"/>
+  <xacro:leg side="right" y="-0.06"/>
   <!-- =============================== -->
   <!-- ROS 2 CONTROL SYSTEM -->
